Commit message: added moveit scene files

File: eusurdf/models/drcbox-valve-bar/model.urdf (robot description, URDF)
Before this commit: robot drcbox-valve-bar, 2 links, 1 joints
Joints:
- joint CRANK-JOINT: origin xyz=0 0 0.353 rpy=0 -0 0  -> xyz=1.13687e-16 0 0.353 rpy=0 -0 0 

File: eusurdf/models/drcbox-valve-large/model.urdf (robot description, URDF)
Before this commit: robot drcbox-valve-large, 2 links, 1 joints
Joints:
- joint CRANK-JOINT: origin xyz=-2.27374e-16 0 0.353 rpy=0 -0 0  -> xyz=0 0 0.353 rpy=0 -0 0 
