Commit message: [textured_models/room73b2-hitachi-fiesta-refrigerator-0/model.urdf] update to more realistic physics parameters

File: eusurdf/textured_models/room73b2-hitachi-fiesta-refrigerator-0/model.urdf (robot description, URDF)
Before this commit: robot room73b2-hitachi-fiesta-refrigerator-0, 7 links, 6 joints
Links:
- link ROOM73B2-HITACHI-FIESTA-REFRIGERATOR-BODYSET2_link: mass 0.001 -> 1.0
- link ROOM73B2-HITACHI-FIESTA-REFRIGERATOR-BODYSET3_link: mass 0.001 -> 1.0
- link ROOM73B2-HITACHI-FIESTA-REFRIGERATOR-BODYSET4_link: mass 0.001 -> 1.0
- link ROOM73B2-HITACHI-FIESTA-REFRIGERATOR-BODYSET5_link: mass 0.001 -> 1.0
- link ROOM73B2-HITACHI-FIESTA-REFRIGERATOR-BODYSET6_link: mass 0.001 -> 1.0
- link ROOM73B2-HITACHI-FIESTA-REFRIGERATOR-BODYSET7_link: mass 0.001 -> 2.0
- link ROOT_link: mass 0.001 -> 50.0
Joints:
- joint DOOR1: limit lower=0 upper=1.5708 effort=100 velocity=0.5 -> lower=0 upper=2.0944 effort=100 velocity=0.5
