Commit message: [textured_models/room73b2-georgia-emerald-mountain-0] add texture of georgia can

File: eusurdf/textured_models/room73b2-georgia-emerald-mountain-0/model.urdf (robot description, URDF)
Before this commit: robot room73b2-georgia-emerald-mountain-0, 1 links, 0 joints
Links:
- link nil_link: mass 0.001 -> 0.3
