Commit message: [eusurdf] parallelize model generation

File: eusurdf/textured_models/room73b2-georgia-emerald-mountain/model.urdf (robot description, URDF)
Before this commit: robot room73b2-iemon-0, 1 links, 0 joints
Links:
- link nil_link: geometry collision mesh filename=model://room73b2-georgia-emerald-mountain/meshes/nil_link_m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 scale=1 1 1; visual mesh filename=model://room73b2-georgia-emerald-mountain/meshes/nil_link_m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 scale=1 1 1

File: eusurdf/textured_models/room73b2-hitachi-fiesta-refrigerator/model.urdf (robot description, URDF)
Before this commit: robot room73b2-hitachi-fiesta-refrigerator-0_static, 7 links, 6 joints
Links:
- link ROOM73B2-HITACHI-FIESTA-REFRIGERATOR-BODYSET2_link: mass 0.001 -> 1.0; geometry collision mesh filename=model://room73b2-hitachi-fiesta-refrigerator/meshes/ROOM73B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 scale=1 1 1; visual mesh filename=model://room73b2-hitachi-fiesta-refrigerator/meshes/ROOM73B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 scale=1 1 1
- link ROOM73B2-HITACHI-FIESTA-REFRIGERATOR-BODYSET3_link: mass 0.001 -> 1.0; geometry collision mesh filename=model://room73b2-hitachi-fiesta-refrigerator/meshes/ROOM73B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 scale=1 1 1; visual mesh filename=model://room73b2-hitachi-fiesta-refrigerator/meshes/ROOM73B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 scale=1 1 1
- link ROOM73B2-HITACHI-FIESTA-REFRIGERATOR-BODYSET4_link: mass 0.001 -> 1.0; geometry collision mesh filename=model://room73b2-hitachi-fiesta-refrigerator/meshes/ROOM73B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 scale=1 1 1; visual mesh filename=model://room73b2-hitachi-fiesta-refrigerator/meshes/ROOM73B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 scale=1 1 1
- link ROOM73B2-HITACHI-FIESTA-REFRIGERATOR-BODYSET5_link: mass 0.001 -> 1.0; geometry collision mesh filename=model://room73b2-hitachi-fiesta-refrigerator/meshes/ROOM73B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 scale=1 1 1; visual mesh filename=model://room73b2-hitachi-fiesta-refrigerator/meshes/ROOM73B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 scale=1 1 1
- link ROOM73B2-HITACHI-FIESTA-REFRIGERATOR-BODYSET6_link: mass 0.001 -> 1.0; geometry collision mesh filename=model://room73b2-hitachi-fiesta-refrigerator/meshes/ROOM73B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 scale=1 1 1; visual mesh filename=model://room73b2-hitachi-fiesta-refrigerator/meshes/ROOM73B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 scale=1 1 1
- link ROOM73B2-HITACHI-FIESTA-REFRIGERATOR-BODYSET7_link: mass 0.001 -> 2.0; geometry collision mesh filename=model://room73b2-hitachi-fiesta-refrigerator/meshes/ROOM73B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 scale=1 1 1; visual mesh filename=model://room73b2-hitachi-fiesta-refrigerator/meshes/ROOM73B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 scale=1 1 1
- link ROOT_link: mass 0.001 -> 50.0; geometry collision mesh filename=model://room73b2-hitachi-fiesta-refrigerator/meshes/ROOT_li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 scale=1 1 1; visual mesh filename=model://room73b2-hitachi-fiesta-refrigerator/meshes/ROOT_li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 scale=1 1 1
Joints:
- joint DOOR1: limit lower=0 upper=1.5708 effort=100 velocity=0.5 -> lower=0 upper=2.0944 effort=100 velocity=0.5

File: eusurdf/textured_models/room73b2-hitachi-fiesta-refrigerator_fixed/model.urdf (robot description, URDF)
Before this commit: robot room73b2-hitachi-fiesta-refrigerator-0, 7 links, 6 joints
Links:
- added link world
- link ROOM73B2-HITACHI-FIESTA-REFRIGERATOR-BODYSET2_link: mass 1.0 -> 0.001; geometry collision mesh filename=model://room73b2-hitachi-fiesta-refrigerator/meshes/ROOM73B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 scale=1 1 1; visual mesh filename=model://room73b2-hitachi-fiesta-refrigerator/meshes/ROOM73B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 scale=1 1 1
- link ROOM73B2-HITACHI-FIESTA-REFRIGERATOR-BODYSET3_link: mass 1.0 -> 0.001; geometry collision mesh filename=model://room73b2-hitachi-fiesta-refrigerator/meshes/ROOM73B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 scale=1 1 1; visual mesh filename=model://room73b2-hitachi-fiesta-refrigerator/meshes/ROOM73B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 scale=1 1 1
- link ROOM73B2-HITACHI-FIESTA-REFRIGERATOR-BODYSET4_link: mass 1.0 -> 0.001; geometry collision mesh filename=model://room73b2-hitachi-fiesta-refrigerator/meshes/ROOM73B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 scale=1 1 1; visual mesh filename=model://room73b2-hitachi-fiesta-refrigerator/meshes/ROOM73B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 scale=1 1 1
- link ROOM73B2-HITACHI-FIESTA-REFRIGERATOR-BODYSET5_link: mass 1.0 -> 0.001; geometry collision mesh filename=model://room73b2-hitachi-fiesta-refrigerator/meshes/ROOM73B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 scale=1 1 1; visual mesh filename=model://room73b2-hitachi-fiesta-refrigerator/meshes/ROOM73B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 scale=1 1 1
- link ROOM73B2-HITACHI-FIESTA-REFRIGERATOR-BODYSET6_link: mass 1.0 -> 0.001; geometry collision mesh filename=model://room73b2-hitachi-fiesta-refrigerator/meshes/ROOM73B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 scale=1 1 1; visual mesh filename=model://room73b2-hitachi-fiesta-refrigerator/meshes/ROOM73B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 scale=1 1 1
- link ROOM73B2-HITACHI-FIESTA-REFRIGERATOR-BODYSET7_link: mass 2.0 -> 0.001; geometry collision mesh filename=model://room73b2-hitachi-fiesta-refrigerator/meshes/ROOM73B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 scale=1 1 1; visual mesh filename=model://room73b2-hitachi-fiesta-refrigerator/meshes/ROOM73B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 scale=1 1 1
- link ROOT_link: mass 50.0 -> 0.001; geometry collision mesh filename=model://room73b2-hitachi-fiesta-refrigerator/meshes/ROOT_li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 scale=1 1 1; visual mesh filename=model://room73b2-hitachi-fiesta-refrigerator/meshes/ROOT_li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 scale=1 1 1
Joints:
- added joint fixed: type fixed, parent world, child ROOT_link
- joint DOOR1: limit lower=0 upper=2.0944 effort=100 velocity=0.5 -> lower=0 upper=1.5708 effort=100 velocity=0.5

File: eusurdf/textured_models/room73b2-hitachi-fiesta-refrigerator_static/model.urdf (robot description, URDF)
Before this commit: robot room73b2-hitachi-fiesta-refrigerator-0_fixed, 8 links, 7 joints
Links:
- removed link world
- link ROOM73B2-HITACHI-FIESTA-REFRIGERATOR-BODYSET2_link: geometry collision mesh filename=model://room73b2-hitachi-fiesta-refrigerator/meshes/ROOM73B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 scale=1 1 1; visual mesh filename=model://room73b2-hitachi-fiesta-refrigerator/meshes/ROOM73B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 scale=1 1 1
- link ROOM73B2-HITACHI-FIESTA-REFRIGERATOR-BODYSET3_link: geometry collision mesh filename=model://room73b2-hitachi-fiesta-refrigerator/meshes/ROOM73B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 scale=1 1 1; visual mesh filename=model://room73b2-hitachi-fiesta-refrigerator/meshes/ROOM73B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 scale=1 1 1
- link ROOM73B2-HITACHI-FIESTA-REFRIGERATOR-BODYSET4_link: geometry collision mesh filename=model://room73b2-hitachi-fiesta-refrigerator/meshes/ROOM73B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 scale=1 1 1; visual mesh filename=model://room73b2-hitachi-fiesta-refrigerator/meshes/ROOM73B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 scale=1 1 1
- link ROOM73B2-HITACHI-FIESTA-REFRIGERATOR-BODYSET5_link: geometry collision mesh filename=model://room73b2-hitachi-fiesta-refrigerator/meshes/ROOM73B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 scale=1 1 1; visual mesh filename=model://room73b2-hitachi-fiesta-refrigerator/meshes/ROOM73B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 scale=1 1 1
- link ROOM73B2-HITACHI-FIESTA-REFRIGERATOR-BODYSET6_link: geometry collision mesh filename=model://room73b2-hitachi-fiesta-refrigerator/meshes/ROOM73B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 scale=1 1 1; visual mesh filename=model://room73b2-hitachi-fiesta-refrigerator/meshes/ROOM73B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 scale=1 1 1
- link ROOM73B2-HITACHI-FIESTA-REFRIGERATOR-BODYSET7_link: geometry collision mesh filename=model://room73b2-hitachi-fiesta-refrigerator/meshes/ROOM73B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 scale=1 1 1; visual mesh filename=model://room73b2-hitachi-fiesta-refrigerator/meshes/ROOM73B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 scale=1 1 1
- link ROOT_link: geometry collision mesh filename=model://room73b2-hitachi-fiesta-refrigerator/meshes/ROOT_li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 scale=1 1 1; visual mesh filename=model://room73b2-hitachi-fiesta-refrigerator/meshes/ROOT_li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 scale=1 1 1
Joints:
- removed joint fixed

File: eusurdf/textured_models/room73b2-iemon/model.urdf (robot description, URDF)
Before this commit: robot room73b2-georgia-emerald-mountain-0_static, 1 links, 0 joints
Links:
- link nil_link: mass 0.001 -> 0.3; geometry collision mesh filename=model://room73b2-iemon/meshes/nil_link_mesh.dae scale=1 1 1; visual mesh filename=model://room73b2-iemon/meshes/nil_link_mesh.dae scale=1 1 1

File: eusurdf/textured_models/room73b2-mac-burger-box/model.urdf (robot description, URDF)
Before this commit: robot room73b2-mac-burger-box-0, 1 links, 0 joints
Links:
- link nil_link: geometry collision mesh filename=model://room73b2-mac-burger-box/meshes/nil_link_mesh.dae scale=1 1 1; visual mesh filename=model://room73b2-mac-burger-box/meshes/nil_link_mesh.dae scale=1 1 1

File: eusurdf/textured_models/room73b2-wanda/model.urdf (robot description, URDF)
Before this commit: robot room73b2-wanda-0, 1 links, 0 joints
Links:
- link nil_link: geometry collision mesh filename=model://room73b2-wanda/meshes/nil_link_mesh.dae scale=1 1 1; visual mesh filename=model://room73b2-wanda/meshes/nil_link_mesh.dae scale=1 1 1
