Commit message: [eusurdf][textured_models] use package://eusurdf instead of model:// for xacro

File: eusurdf/textured_models/room73b2-georgia-emerald-mountain/model.urdf.xacro (robot description, xacro)
@@ -9,5 +9,5 @@
         <origin xyz="0 0 0" rpy="0 -0 0"/>
         <geometry>
-          <mesh filename="model://room73b2-georgia-emerald-mountain/meshes/nil_link_mesh.dae" scale="1 1 1"/>
+          <mesh filename="package://eusurdf/textured_models/room73b2-georgia-emerald-mountain/meshes/nil_link_mesh.dae" scale="1 1 1"/>
         </geometry>
       </visual>
@@ -15,5 +15,5 @@
         <origin xyz="0 0 0" rpy="0 -0 0"/>
         <geometry>
-          <mesh filename="model://room73b2-georgia-emerald-mountain/meshes/nil_link_mesh.dae" scale="1 1 1"/>
+          <mesh filename="package://eusurdf/textured_models/room73b2-georgia-emerald-mountain/meshes/nil_link_mesh.dae" scale="1 1 1"/>
         </geometry>
       </collision>

File: eusurdf/textured_models/room73b2-hitachi-fiesta-refrigerator/model.urdf.xacro (robot description, xacro)
@@ -9,11 +9,11 @@
         <origin xyz="0 0 0" rpy="0 -0 0"/>
         <geometry>
-          <mesh filename="model://room73b2-hitachi-fiesta-refrigerator/meshes/ROOT_link_mesh.dae" scale="1 1 1"/>
-        </geometry>
-      </visual>
-      <collision>
-        <origin xyz="0 0 0" rpy="0 -0 0"/>
-        <geometry>
-          <mesh filename="model://room73b2-hitachi-fiesta-refrigerator/meshes/ROOT_link_mesh.dae" scale="1 1 1"/>
+          <mesh filename="package://eusurdf/textured_models/room73b2-hitachi-fiesta-refrigerator/meshes/ROOT_link_mesh.dae" scale="1 1 1"/>
+        </geometry>
+      </visual>
+      <collision>
+        <origin xyz="0 0 0" rpy="0 -0 0"/>
+        <geometry>
+          <mesh filename="package://eusurdf/textured_models/room73b2-hitachi-fiesta-refrigerator/meshes/ROOT_link_mesh.dae" scale="1 1 1"/>
         </geometry>
       </collision>
@@ -32,5 +32,5 @@
         <origin xyz="0.3 0.245 0.85" rpy="-1.57 -0 0"/>
         <geometry>
-          <mesh filename="model://room73b2-hitachi-fiesta-refrigerator/meshes/ROOM73B2-HITACHI-FIESTA-REFRIGERATOR-BODYSET7_link_mesh.dae" scale="1 1 1"/>
+          <mesh filename="package://eusurdf/textured_models/room73b2-hitachi-fiesta-refrigerator/meshes/ROOM73B2-HITACHI-FIESTA-REFRIGERATOR-BODYSET7_link_mesh.dae" scale="1 1 1"/>
         </geometry>
       </visual>
@@ -38,5 +38,5 @@
         <origin xyz="0.3 0.245 0.85" rpy="-1.57 -0 0"/>
         <geometry>
-          <mesh filename="model://room73b2-hitachi-fiesta-refrigerator/meshes/ROOM73B2-HITACHI-FIESTA-REFRIGERATOR-BODYSET7_link_mesh.dae" scale="1 1 1"/>
+          <mesh filename="package://eusurdf/textured_models/room73b2-hitachi-fiesta-refrigerator/meshes/ROOM73B2-HITACHI-FIESTA-REFRIGERATOR-BODYSET7_link_mesh.dae" scale="1 1 1"/>
         </geometry>
       </collision>
@@ -55,5 +55,5 @@
         <origin xyz="0.05 0 0.66" rpy="0 -0 0"/>
         <geometry>
-          <mesh filename="model://room73b2-hitachi-fiesta-refrigerator/meshes/ROOM73B2-HITACHI-FIESTA-REFRIGERATOR-BODYSET6_link_mesh.dae" scale="1 1 1"/>
+          <mesh filename="package://eusurdf/textured_models/room73b2-hitachi-fiesta-refrigerator/meshes/ROOM73B2-HITACHI-FIESTA-REFRIGERATOR-BODYSET6_link_mesh.dae" scale="1 1 1"/>
         </geometry>
       </visual>
@@ -61,5 +61,5 @@
         <origin xyz="0.05 0 0.66" rpy="0 -0 0"/>
         <geometry>
-          <mesh filename="model://room73b2-hitachi-fiesta-refrigerator/meshes/ROOM73B2-HITACHI-FIESTA-REFRIGERATOR-BODYSET6_link_mesh.dae" scale="1 1 1"/>
+          <mesh filename="package://eusurdf/textured_models/room73b2-hitachi-fiesta-refrigerator/meshes/ROOM73B2-HITACHI-FIESTA-REFRIGERATOR-BODYSET6_link_mesh.dae" scale="1 1 1"/>
         </geometry>
       </collision>
@@ -78,5 +78,5 @@
         <origin xyz="0.06 0 0.24" rpy="0 -0 0"/>
         <geometry>
-          <mesh filename="model://room73b2-hitachi-fiesta-refrigerator/meshes/ROOM73B2-HITACHI-FIESTA-REFRIGERATOR-BODYSET5_link_mesh.dae" scale="1 1 1"/>
+          <mesh filename="package://eusurdf/textured_models/room73b2-hitachi-fiesta-refrigerator/meshes/ROOM73B2-HITACHI-FIESTA-REFRIGERATOR-BODYSET5_link_mesh.dae" scale="1 1 1"/>
         </geometry>
       </visual>
@@ -84,5 +84,5 @@
         <origin xyz="0.06 0 0.24" rpy="0 -0 0"/>
         <geometry>
-          <mesh filename="model://room73b2-hitachi-fiesta-refrigerator/meshes/ROOM73B2-HITACHI-FIESTA-REFRIGERATOR-BODYSET5_link_mesh.dae" scale="1 1 1"/>
+          <mesh filename="package://eusurdf/textured_models/room73b2-hitachi-fiesta-refrigerator/meshes/ROOM73B2-HITACHI-FIESTA-REFRIGERATOR-BODYSET5_link_mesh.dae" scale="1 1 1"/>
         </geometry>
       </collision>
@@ -101,5 +101,5 @@
         <origin xyz="-0.095 0 1.275" rpy="0 -0 0"/>
         <geometry>
-          <mesh filename="model://room73b2-hitachi-fiesta-refrigerator/meshes/ROOM73B2-HITACHI-FIESTA-REFRIGERATOR-BODYSET4_link_mesh.dae" scale="1 1 1"/>
+          <mesh filename="package://eusurdf/textured_models/room73b2-hitachi-fiesta-refrigerator/meshes/ROOM73B2-HITACHI-FIESTA-REFRIGERATOR-BODYSET4_link_mesh.dae" scale="1 1 1"/>
         </geometry>
       </visual>
@@ -107,5 +107,5 @@
         <origin xyz="-0.095 0 1.275" rpy="0 -0 0"/>
         <geometry>
-          <mesh filename="model://room73b2-hitachi-fiesta-refrigerator/meshes/ROOM73B2-HITACHI-FIESTA-REFRIGERATOR-BODYSET4_link_mesh.dae" scale="1 1 1"/>
+          <mesh filename="package://eusurdf/textured_models/room73b2-hitachi-fiesta-refrigerator/meshes/ROOM73B2-HITACHI-FIESTA-REFRIGERATOR-BODYSET4_link_mesh.dae" scale="1 1 1"/>
         </geometry>
       </collision>
@@ -124,5 +124,5 @@
         <origin xyz="-0.095 0 1.085" rpy="0 -0 0"/>
         <geometry>
-          <mesh filename="model://room73b2-hitachi-fiesta-refrigerator/meshes/ROOM73B2-HITACHI-FIESTA-REFRIGERATOR-BODYSET3_link_mesh.dae" scale="1 1 1"/>
+          <mesh filename="package://eusurdf/textured_models/room73b2-hitachi-fiesta-refrigerator/meshes/ROOM73B2-HITACHI-FIESTA-REFRIGERATOR-BODYSET3_link_mesh.dae" scale="1 1 1"/>
         </geometry>
       </visual>
@@ -130,5 +130,5 @@
         <origin xyz="-0.095 0 1.085" rpy="0 -0 0"/>
         <geometry>
-          <mesh filename="model://room73b2-hitachi-fiesta-refrigerator/meshes/ROOM73B2-HITACHI-FIESTA-REFRIGERATOR-BODYSET3_link_mesh.dae" scale="1 1 1"/>
+          <mesh filename="package://eusurdf/textured_models/room73b2-hitachi-fiesta-refrigerator/meshes/ROOM73B2-HITACHI-FIESTA-REFRIGERATOR-BODYSET3_link_mesh.dae" scale="1 1 1"/>
         </geometry>
       </collision>
@@ -147,5 +147,5 @@
         <origin xyz="-0.095 0 0.935" rpy="0 -0 0"/>
         <geometry>
-          <mesh filename="model://room73b2-hitachi-fiesta-refrigerator/meshes/ROOM73B2-HITACHI-FIESTA-REFRIGERATOR-BODYSET2_link_mesh.dae" scale="1 1 1"/>
+          <mesh filename="package://eusurdf/textured_models/room73b2-hitachi-fiesta-refrigerator/meshes/ROOM73B2-HITACHI-FIESTA-REFRIGERATOR-BODYSET2_link_mesh.dae" scale="1 1 1"/>
         </geometry>
       </visual>
@@ -153,5 +153,5 @@
         <origin xyz="-0.095 0 0.935" rpy="0 -0 0"/>
         <geometry>
-          <mesh filename="model://room73b2-hitachi-fiesta-refrigerator/meshes/ROOM73B2-HITACHI-FIESTA-REFRIGERATOR-BODYSET2_link_mesh.dae" scale="1 1 1"/>
+          <mesh filename="package://eusurdf/textured_models/room73b2-hitachi-fiesta-refrigerator/meshes/ROOM73B2-HITACHI-FIESTA-REFRIGERATOR-BODYSET2_link_mesh.dae" scale="1 1 1"/>
         </geometry>
       </collision>

File: eusurdf/textured_models/room73b2-hitachi-fiesta-refrigerator_fixed/model.urdf.xacro (robot description, xacro)
@@ -9,11 +9,11 @@
         <origin xyz="0 0 0" rpy="0 -0 0"/>
         <geometry>
-          <mesh filename="model://room73b2-hitachi-fiesta-refrigerator/meshes/ROOT_link_mesh.dae" scale="1 1 1"/>
-        </geometry>
-      </visual>
-      <collision>
-        <origin xyz="0 0 0" rpy="0 -0 0"/>
-        <geometry>
-          <mesh filename="model://room73b2-hitachi-fiesta-refrigerator/meshes/ROOT_link_mesh.dae" scale="1 1 1"/>
+          <mesh filename="package://eusurdf/textured_models/room73b2-hitachi-fiesta-refrigerator/meshes/ROOT_link_mesh.dae" scale="1 1 1"/>
+        </geometry>
+      </visual>
+      <collision>
+        <origin xyz="0 0 0" rpy="0 -0 0"/>
+        <geometry>
+          <mesh filename="package://eusurdf/textured_models/room73b2-hitachi-fiesta-refrigerator/meshes/ROOT_link_mesh.dae" scale="1 1 1"/>
         </geometry>
       </collision>
@@ -32,5 +32,5 @@
         <origin xyz="0.3 0.25 0.85" rpy="-1.57 -0 0"/>
         <geometry>
-          <mesh filename="model://room73b2-hitachi-fiesta-refrigerator/meshes/ROOM73B2-HITACHI-FIESTA-REFRIGERATOR-BODYSET7_link_mesh.dae" scale="1 1 1"/>
+          <mesh filename="package://eusurdf/textured_models/room73b2-hitachi-fiesta-refrigerator/meshes/ROOM73B2-HITACHI-FIESTA-REFRIGERATOR-BODYSET7_link_mesh.dae" scale="1 1 1"/>
         </geometry>
       </visual>
@@ -38,5 +38,5 @@
         <origin xyz="0.3 0.245 0.85" rpy="-1.57 -0 0"/>
         <geometry>
-          <mesh filename="model://room73b2-hitachi-fiesta-refrigerator/meshes/ROOM73B2-HITACHI-FIESTA-REFRIGERATOR-BODYSET7_link_mesh.dae" scale="1 1 1"/>
+          <mesh filename="package://eusurdf/textured_models/room73b2-hitachi-fiesta-refrigerator/meshes/ROOM73B2-HITACHI-FIESTA-REFRIGERATOR-BODYSET7_link_mesh.dae" scale="1 1 1"/>
         </geometry>
       </collision>
@@ -55,5 +55,5 @@
         <origin xyz="0.05 0 0.66" rpy="0 -0 0"/>
         <geometry>
-          <mesh filename="model://room73b2-hitachi-fiesta-refrigerator/meshes/ROOM73B2-HITACHI-FIESTA-REFRIGERATOR-BODYSET6_link_mesh.dae" scale="1 1 1"/>
+          <mesh filename="package://eusurdf/textured_models/room73b2-hitachi-fiesta-refrigerator/meshes/ROOM73B2-HITACHI-FIESTA-REFRIGERATOR-BODYSET6_link_mesh.dae" scale="1 1 1"/>
         </geometry>
       </visual>
@@ -61,5 +61,5 @@
         <origin xyz="0.05 0 0.66" rpy="0 -0 0"/>
         <geometry>
-          <mesh filename="model://room73b2-hitachi-fiesta-refrigerator/meshes/ROOM73B2-HITACHI-FIESTA-REFRIGERATOR-BODYSET6_link_mesh.dae" scale="1 1 1"/>
+          <mesh filename="package://eusurdf/textured_models/room73b2-hitachi-fiesta-refrigerator/meshes/ROOM73B2-HITACHI-FIESTA-REFRIGERATOR-BODYSET6_link_mesh.dae" scale="1 1 1"/>
         </geometry>
       </collision>
@@ -78,5 +78,5 @@
         <origin xyz="0.06 0 0.24" rpy="0 -0 0"/>
         <geometry>
-          <mesh filename="model://room73b2-hitachi-fiesta-refrigerator/meshes/ROOM73B2-HITACHI-FIESTA-REFRIGERATOR-BODYSET5_link_mesh.dae" scale="1 1 1"/>
+          <mesh filename="package://eusurdf/textured_models/room73b2-hitachi-fiesta-refrigerator/meshes/ROOM73B2-HITACHI-FIESTA-REFRIGERATOR-BODYSET5_link_mesh.dae" scale="1 1 1"/>
         </geometry>
       </visual>
@@ -84,5 +84,5 @@
         <origin xyz="0.06 0 0.24" rpy="0 -0 0"/>
         <geometry>
-          <mesh filename="model://room73b2-hitachi-fiesta-refrigerator/meshes/ROOM73B2-HITACHI-FIESTA-REFRIGERATOR-BODYSET5_link_mesh.dae" scale="1 1 1"/>
+          <mesh filename="package://eusurdf/textured_models/room73b2-hitachi-fiesta-refrigerator/meshes/ROOM73B2-HITACHI-FIESTA-REFRIGERATOR-BODYSET5_link_mesh.dae" scale="1 1 1"/>
         </geometry>
       </collision>
@@ -101,5 +101,5 @@
         <origin xyz="-0.095 0 1.275" rpy="0 -0 0"/>
         <geometry>
-          <mesh filename="model://room73b2-hitachi-fiesta-refrigerator/meshes/ROOM73B2-HITACHI-FIESTA-REFRIGERATOR-BODYSET4_link_mesh.dae" scale="1 1 1"/>
+          <mesh filename="package://eusurdf/textured_models/room73b2-hitachi-fiesta-refrigerator/meshes/ROOM73B2-HITACHI-FIESTA-REFRIGERATOR-BODYSET4_link_mesh.dae" scale="1 1 1"/>
         </geometry>
       </visual>
@@ -107,5 +107,5 @@
         <origin xyz="-0.095 0 1.275" rpy="0 -0 0"/>
         <geometry>
-          <mesh filename="model://room73b2-hitachi-fiesta-refrigerator/meshes/ROOM73B2-HITACHI-FIESTA-REFRIGERATOR-BODYSET4_link_mesh.dae" scale="1 1 1"/>
+          <mesh filename="package://eusurdf/textured_models/room73b2-hitachi-fiesta-refrigerator/meshes/ROOM73B2-HITACHI-FIESTA-REFRIGERATOR-BODYSET4_link_mesh.dae" scale="1 1 1"/>
         </geometry>
       </collision>
@@ -124,5 +124,5 @@
         <origin xyz="-0.095 0 1.085" rpy="0 -0 0"/>
         <geometry>
-          <mesh filename="model://room73b2-hitachi-fiesta-refrigerator/meshes/ROOM73B2-HITACHI-FIESTA-REFRIGERATOR-BODYSET3_link_mesh.dae" scale="1 1 1"/>
+          <mesh filename="package://eusurdf/textured_models/room73b2-hitachi-fiesta-refrigerator/meshes/ROOM73B2-HITACHI-FIESTA-REFRIGERATOR-BODYSET3_link_mesh.dae" scale="1 1 1"/>
         </geometry>
       </visual>
@@ -130,5 +130,5 @@
         <origin xyz="-0.095 0 1.085" rpy="0 -0 0"/>
         <geometry>
-          <mesh filename="model://room73b2-hitachi-fiesta-refrigerator/meshes/ROOM73B2-HITACHI-FIESTA-REFRIGERATOR-BODYSET3_link_mesh.dae" scale="1 1 1"/>
+          <mesh filename="package://eusurdf/textured_models/room73b2-hitachi-fiesta-refrigerator/meshes/ROOM73B2-HITACHI-FIESTA-REFRIGERATOR-BODYSET3_link_mesh.dae" scale="1 1 1"/>
         </geometry>
       </collision>
@@ -147,5 +147,5 @@
         <origin xyz="-0.095 0 0.935" rpy="0 -0 0"/>
         <geometry>
-          <mesh filename="model://room73b2-hitachi-fiesta-refrigerator/meshes/ROOM73B2-HITACHI-FIESTA-REFRIGERATOR-BODYSET2_link_mesh.dae" scale="1 1 1"/>
+          <mesh filename="package://eusurdf/textured_models/room73b2-hitachi-fiesta-refrigerator/meshes/ROOM73B2-HITACHI-FIESTA-REFRIGERATOR-BODYSET2_link_mesh.dae" scale="1 1 1"/>
         </geometry>
       </visual>
@@ -153,5 +153,5 @@
         <origin xyz="-0.095 0 0.935" rpy="0 -0 0"/>
         <geometry>
-          <mesh filename="model://room73b2-hitachi-fiesta-refrigerator/meshes/ROOM73B2-HITACHI-FIESTA-REFRIGERATOR-BODYSET2_link_mesh.dae" scale="1 1 1"/>
+          <mesh filename="package://eusurdf/textured_models/room73b2-hitachi-fiesta-refrigerator/meshes/ROOM73B2-HITACHI-FIESTA-REFRIGERATOR-BODYSET2_link_mesh.dae" scale="1 1 1"/>
         </geometry>
       </collision>

File: eusurdf/textured_models/room73b2-hitachi-fiesta-refrigerator_static/model.urdf.xacro (robot description, xacro)
@@ -9,11 +9,11 @@
         <origin xyz="0 0 0" rpy="0 -0 0"/>
         <geometry>
-          <mesh filename="model://room73b2-hitachi-fiesta-refrigerator/meshes/ROOT_link_mesh.dae" scale="1 1 1"/>
-        </geometry>
-      </visual>
-      <collision>
-        <origin xyz="0 0 0" rpy="0 -0 0"/>
-        <geometry>
-          <mesh filename="model://room73b2-hitachi-fiesta-refrigerator/meshes/ROOT_link_mesh.dae" scale="1 1 1"/>
+          <mesh filename="package://eusurdf/textured_models/room73b2-hitachi-fiesta-refrigerator/meshes/ROOT_link_mesh.dae" scale="1 1 1"/>
+        </geometry>
+      </visual>
+      <collision>
+        <origin xyz="0 0 0" rpy="0 -0 0"/>
+        <geometry>
+          <mesh filename="package://eusurdf/textured_models/room73b2-hitachi-fiesta-refrigerator/meshes/ROOT_link_mesh.dae" scale="1 1 1"/>
         </geometry>
       </collision>
@@ -32,5 +32,5 @@
         <origin xyz="0.3 0.245 0.85" rpy="-1.57 -0 0"/>
         <geometry>
-          <mesh filename="model://room73b2-hitachi-fiesta-refrigerator/meshes/ROOM73B2-HITACHI-FIESTA-REFRIGERATOR-BODYSET7_link_mesh.dae" scale="1 1 1"/>
+          <mesh filename="package://eusurdf/textured_models/room73b2-hitachi-fiesta-refrigerator/meshes/ROOM73B2-HITACHI-FIESTA-REFRIGERATOR-BODYSET7_link_mesh.dae" scale="1 1 1"/>
         </geometry>
       </visual>
@@ -38,5 +38,5 @@
         <origin xyz="0.3 0.245 0.85" rpy="-1.57 -0 0"/>
         <geometry>
-          <mesh filename="model://room73b2-hitachi-fiesta-refrigerator/meshes/ROOM73B2-HITACHI-FIESTA-REFRIGERATOR-BODYSET7_link_mesh.dae" scale="1 1 1"/>
+          <mesh filename="package://eusurdf/textured_models/room73b2-hitachi-fiesta-refrigerator/meshes/ROOM73B2-HITACHI-FIESTA-REFRIGERATOR-BODYSET7_link_mesh.dae" scale="1 1 1"/>
         </geometry>
       </collision>
@@ -55,5 +55,5 @@
         <origin xyz="0.05 0 0.66" rpy="0 -0 0"/>
         <geometry>
-          <mesh filename="model://room73b2-hitachi-fiesta-refrigerator/meshes/ROOM73B2-HITACHI-FIESTA-REFRIGERATOR-BODYSET6_link_mesh.dae" scale="1 1 1"/>
+          <mesh filename="package://eusurdf/textured_models/room73b2-hitachi-fiesta-refrigerator/meshes/ROOM73B2-HITACHI-FIESTA-REFRIGERATOR-BODYSET6_link_mesh.dae" scale="1 1 1"/>
         </geometry>
       </visual>
@@ -61,5 +61,5 @@
         <origin xyz="0.05 0 0.66" rpy="0 -0 0"/>
         <geometry>
-          <mesh filename="model://room73b2-hitachi-fiesta-refrigerator/meshes/ROOM73B2-HITACHI-FIESTA-REFRIGERATOR-BODYSET6_link_mesh.dae" scale="1 1 1"/>
+          <mesh filename="package://eusurdf/textured_models/room73b2-hitachi-fiesta-refrigerator/meshes/ROOM73B2-HITACHI-FIESTA-REFRIGERATOR-BODYSET6_link_mesh.dae" scale="1 1 1"/>
         </geometry>
       </collision>
@@ -78,5 +78,5 @@
         <origin xyz="0.06 0 0.24" rpy="0 -0 0"/>
         <geometry>
-          <mesh filename="model://room73b2-hitachi-fiesta-refrigerator/meshes/ROOM73B2-HITACHI-FIESTA-REFRIGERATOR-BODYSET5_link_mesh.dae" scale="1 1 1"/>
+          <mesh filename="package://eusurdf/textured_models/room73b2-hitachi-fiesta-refrigerator/meshes/ROOM73B2-HITACHI-FIESTA-REFRIGERATOR-BODYSET5_link_mesh.dae" scale="1 1 1"/>
         </geometry>
       </visual>
@@ -84,5 +84,5 @@
         <origin xyz="0.06 0 0.24" rpy="0 -0 0"/>
         <geometry>
-          <mesh filename="model://room73b2-hitachi-fiesta-refrigerator/meshes/ROOM73B2-HITACHI-FIESTA-REFRIGERATOR-BODYSET5_link_mesh.dae" scale="1 1 1"/>
+          <mesh filename="package://eusurdf/textured_models/room73b2-hitachi-fiesta-refrigerator/meshes/ROOM73B2-HITACHI-FIESTA-REFRIGERATOR-BODYSET5_link_mesh.dae" scale="1 1 1"/>
         </geometry>
       </collision>
@@ -101,5 +101,5 @@
         <origin xyz="-0.095 0 1.275" rpy="0 -0 0"/>
         <geometry>
-          <mesh filename="model://room73b2-hitachi-fiesta-refrigerator/meshes/ROOM73B2-HITACHI-FIESTA-REFRIGERATOR-BODYSET4_link_mesh.dae" scale="1 1 1"/>
+          <mesh filename="package://eusurdf/textured_models/room73b2-hitachi-fiesta-refrigerator/meshes/ROOM73B2-HITACHI-FIESTA-REFRIGERATOR-BODYSET4_link_mesh.dae" scale="1 1 1"/>
         </geometry>
       </visual>
@@ -107,5 +107,5 @@
         <origin xyz="-0.095 0 1.275" rpy="0 -0 0"/>
         <geometry>
-          <mesh filename="model://room73b2-hitachi-fiesta-refrigerator/meshes/ROOM73B2-HITACHI-FIESTA-REFRIGERATOR-BODYSET4_link_mesh.dae" scale="1 1 1"/>
+          <mesh filename="package://eusurdf/textured_models/room73b2-hitachi-fiesta-refrigerator/meshes/ROOM73B2-HITACHI-FIESTA-REFRIGERATOR-BODYSET4_link_mesh.dae" scale="1 1 1"/>
         </geometry>
       </collision>
@@ -124,5 +124,5 @@
         <origin xyz="-0.095 0 1.085" rpy="0 -0 0"/>
         <geometry>
-          <mesh filename="model://room73b2-hitachi-fiesta-refrigerator/meshes/ROOM73B2-HITACHI-FIESTA-REFRIGERATOR-BODYSET3_link_mesh.dae" scale="1 1 1"/>
+          <mesh filename="package://eusurdf/textured_models/room73b2-hitachi-fiesta-refrigerator/meshes/ROOM73B2-HITACHI-FIESTA-REFRIGERATOR-BODYSET3_link_mesh.dae" scale="1 1 1"/>
         </geometry>
       </visual>
@@ -130,5 +130,5 @@
         <origin xyz="-0.095 0 1.085" rpy="0 -0 0"/>
         <geometry>
-          <mesh filename="model://room73b2-hitachi-fiesta-refrigerator/meshes/ROOM73B2-HITACHI-FIESTA-REFRIGERATOR-BODYSET3_link_mesh.dae" scale="1 1 1"/>
+          <mesh filename="package://eusurdf/textured_models/room73b2-hitachi-fiesta-refrigerator/meshes/ROOM73B2-HITACHI-FIESTA-REFRIGERATOR-BODYSET3_link_mesh.dae" scale="1 1 1"/>
         </geometry>
       </collision>
@@ -147,5 +147,5 @@
         <origin xyz="-0.095 0 0.935" rpy="0 -0 0"/>
         <geometry>
-          <mesh filename="model://room73b2-hitachi-fiesta-refrigerator/meshes/ROOM73B2-HITACHI-FIESTA-REFRIGERATOR-BODYSET2_link_mesh.dae" scale="1 1 1"/>
+          <mesh filename="package://eusurdf/textured_models/room73b2-hitachi-fiesta-refrigerator/meshes/ROOM73B2-HITACHI-FIESTA-REFRIGERATOR-BODYSET2_link_mesh.dae" scale="1 1 1"/>
         </geometry>
       </visual>
@@ -153,5 +153,5 @@
         <origin xyz="-0.095 0 0.935" rpy="0 -0 0"/>
         <geometry>
-          <mesh filename="model://room73b2-hitachi-fiesta-refrigerator/meshes/ROOM73B2-HITACHI-FIESTA-REFRIGERATOR-BODYSET2_link_mesh.dae" scale="1 1 1"/>
+          <mesh filename="package://eusurdf/textured_models/room73b2-hitachi-fiesta-refrigerator/meshes/ROOM73B2-HITACHI-FIESTA-REFRIGERATOR-BODYSET2_link_mesh.dae" scale="1 1 1"/>
         </geometry>
       </collision>

File: eusurdf/textured_models/room73b2-iemon/model.urdf.xacro (robot description, xacro)
@@ -9,5 +9,5 @@
         <origin xyz="0 0 0" rpy="0 -0 0"/>
         <geometry>
-          <mesh filename="model://room73b2-iemon/meshes/nil_link_mesh.dae" scale="1 1 1"/>
+          <mesh filename="package://eusurdf/textured_models/room73b2-iemon/meshes/nil_link_mesh.dae" scale="1 1 1"/>
         </geometry>
       </visual>
@@ -15,5 +15,5 @@
         <origin xyz="0 0 0" rpy="0 -0 0"/>
         <geometry>
-          <mesh filename="model://room73b2-iemon/meshes/nil_link_mesh.dae" scale="1 1 1"/>
+          <mesh filename="package://eusurdf/textured_models/room73b2-iemon/meshes/nil_link_mesh.dae" scale="1 1 1"/>
         </geometry>
       </collision>

File: eusurdf/textured_models/room73b2-mac-burger-box/model.urdf.xacro (robot description, xacro)
@@ -9,5 +9,5 @@
         <origin xyz="0 0 0" rpy="0 -0 0"/>
         <geometry>
-          <mesh filename="model://room73b2-mac-burger-box/meshes/nil_link_mesh.dae" scale="1 1 1"/>
+          <mesh filename="package://eusurdf/textured_models/room73b2-mac-burger-box/meshes/nil_link_mesh.dae" scale="1 1 1"/>
         </geometry>
       </visual>
@@ -15,5 +15,5 @@
         <origin xyz="0 0 0" rpy="0 -0 0"/>
         <geometry>
-          <mesh filename="model://room73b2-mac-burger-box/meshes/nil_link_mesh.dae" scale="1 1 1"/>
+          <mesh filename="package://eusurdf/textured_models/room73b2-mac-burger-box/meshes/nil_link_mesh.dae" scale="1 1 1"/>
         </geometry>
       </collision>

File: eusurdf/textured_models/room73b2-wanda/model.urdf.xacro (robot description, xacro)
@@ -9,5 +9,5 @@
         <origin xyz="0 0 0" rpy="0 -0 0"/>
         <geometry>
-          <mesh filename="model://room73b2-wanda/meshes/nil_link_mesh.dae" scale="1 1 1"/>
+          <mesh filename="package://eusurdf/textured_models/room73b2-wanda/meshes/nil_link_mesh.dae" scale="1 1 1"/>
         </geometry>
       </visual>
@@ -15,5 +15,5 @@
         <origin xyz="0 0 0" rpy="0 -0 0"/>
         <geometry>
-          <mesh filename="model://room73b2-wanda/meshes/nil_link_mesh.dae" scale="1 1 1"/>
+          <mesh filename="package://eusurdf/textured_models/room73b2-wanda/meshes/nil_link_mesh.dae" scale="1 1 1"/>
         </geometry>
       </collision>
